Commit message: placed arm on platform and added camera

File: model/arm.urdf.xacro (robot description, xacro)
@@ -2,4 +2,5 @@
 <robot name="robot" xmlns:xacro="http://ros.org/wiki/xacro">
     <xacro:include filename="$(find mobile_robot)/model/arm.gazebo"/>
+<!--
     <link name="world">
     </link>
@@ -8,5 +9,5 @@
         <child link="base_link"/>
         <origin xyz="1 1 0" rpy="0 0 0"/>
-    </joint>
+    </joint> -->
     <link name="base_link">
         <visual>
@@ -27,6 +28,6 @@
         <inertial>
         <mass value="1.0"/> <!-- Mass of the link in kilograms -->
-        <origin xyz="0 0 0.005" rpy="0 0 0"/> <!-- Center of mass relative to the link frame -->
-        <inertia ixx="0.001" ixy="0" ixz="0" iyy="0.001" iyz="0" izz="0.001"/> <!-- Inertia tensor components -->
+        <origin xyz="0 0 0.08" rpy="0 0 0"/> <!-- Center of mass relative to the link frame -->
+        <inertia ixx="0.00398" ixy="0" ixz="0" iyy="0.00398" iyz="0" izz="0.00370"/> <!-- Inertia tensor components -->
         </inertial>
     </link>
@@ -54,7 +55,7 @@
     </collision>
     <inertial>
-      <mass value="1.0"/> <!-- Mass of the link in kilograms -->
-      <origin xyz="0 0 0" rpy="0 0 0"/> <!-- Center of mass relative to the link frame -->
-      <inertia ixx="0.001" ixy="0" ixz="0" iyy="0.001" iyz="0" izz="0.001"/> <!-- Inertia tensor components -->
+      <mass value="2.0"/> <!-- Mass of the link in kilograms -->
+      <origin xyz="0 0 0.065" rpy="0 0 0"/> <!-- Center of mass relative to the link frame, centered along height -->
+      <inertia ixx="0.00462" ixy="0" ixz="0" iyy="0.00462" iyz="0" izz="0.00360"/> <!-- Updated Inertia tensor components -->
     </inertial>
   </link>
@@ -82,7 +83,7 @@
     </collision>
     <inertial>
-      <mass value="1.0"/> <!-- Mass of the link in kilograms -->
-      <origin xyz="0 0 0" rpy="0 0 0"/> <!-- Center of mass relative to the link frame -->
-      <inertia ixx="0.001" ixy="0" ixz="0" iyy="0.001" iyz="0" izz="0.001"/> <!-- Inertia tensor components -->
+      <mass value="2.0"/> <!-- Mass of the link in kilograms -->
+      <origin xyz="0 0.34 0" rpy="0 0 0"/> <!-- Center of mass is offset along the y-axis (half the length of the cylinder) -->
+      <inertia ixx="0.07817" ixy="0" ixz="0" iyy="0.07817" iyz="0" izz="0.00221"/> <!-- Updated Inertia tensor components -->
     </inertial>
   </link>
@@ -110,9 +111,10 @@
     </collision>
     <inertial>
-      <mass value="1.0"/> <!-- Mass of the link in kilograms -->
-      <origin xyz="0 0 0" rpy="0 0 0"/> <!-- Center of mass relative to the link frame -->
-      <inertia ixx="0.001" ixy="0" ixz="0" iyy="0.001" iyz="0" izz="0.001"/> <!-- Inertia tensor components -->
+        <mass value="1.0"/> <!-- Mass of the link in kilograms -->
+        <origin xyz="0 0.21 0" rpy="0 0 0"/> <!-- Center of mass relative to the link frame, centered along height -->
+        <inertia ixx="0.01506" ixy="0" ixz="0" iyy="0.01506" iyz="0" izz="0.000722"/> <!-- Updated Inertia tensor components -->
     </inertial>
   </link>
+  <xacro:include filename="$(find mobile_robot)/model/camera.xacro"/>
   <ros2_control name="GazeboSimSystem" type="system">
     <hardware>
@@ -129,5 +131,5 @@
         <command_interface name="position"/>
         <state_interface name="position">
-            <param name="initial_value">1.0</param>
+            <param name="initial_value">0.0</param>
         </state_interface>
         <state_interface name="velocity"/>

File: model/platform.xacro (robot description, xacro)
@@ -8,5 +8,5 @@
 <xacro:property name="body_link_x_dim" value="1"/>
 <xacro:property name="body_link_y_dim" value="0.6"/>
-<xacro:property name="body_link_z_dim" value="0.3"/>
+<xacro:property name="body_link_z_dim" value="0.2"/>
 <!-- Wheel dimenstions -->
 <xacro:property name="wheel_link_rad" value="0.15"/>
